File: Hardware/MiniMoto.brd (EAGLE design)
At the start: 25.4 x 25.4 mm, 23 parts, among them J1 M02PTH3, J2 M023.5MM, J3 M02PTH3, J4 M023.5MM, J5 M02PTH3, J6 M023.5MM, J7 M04X2, U1 DRV8830

Commit message: Tweaks for release, add lib
Other:
- board text added: "v10"
- board text removed: "v01"
Changed lines of the file:
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@@
 <layer number="39" name="tKeepout" color="4" fill="11" visible="no" active="yes"/>
 <layer number="40" name="bKeepout" color="1" fill="11" visible="no" active="yes"/>
-<layer number="41" name="tRestrict" color="4" fill="10" visible="yes" active="yes"/>
+<layer number="41" name="tRestrict" color="4" fill="10" visible="no" active="yes"/>
 <layer number="42" name="bRestrict" color="1" fill="10" visible="no" active="yes"/>
+<layer number="43" name="vRestrict" color="2" fill="10" visible="no" active="yes"/>
 <layer number="44" name="Drills" color="7" fill="1" visible="no" active="yes"/>
 <layer number="45" name="Holes" color="7" fill="1" visible="yes" active="yes"/>
@@
 <layer number="37" name="tTest" color="7" fill="1" visible="no" active="no"/>
 <layer number="38" name="bTest" color="7" fill="1" visible="no" active="no"/>
-<layer number="43" name="vRestrict" color="2" fill="10" visible="no" active="no"/>
 <layer number="47" name="Measures" color="7" fill="1" visible="no" active="no"/>
 <layer number="48" name="Document" color="7" fill="1" visible="no" active="no"/>
@@
 <text x="10.033" y="23.241" size="1.27" layer="21" font="vector" ratio="15" align="bottom-center">MiniMoto</text>
 <text x="21.336" y="13.97" size="1.27" layer="22" font="vector" ratio="15" rot="MR90" align="bottom-center">MiniMoto</text>
-<text x="1.905" y="15.748" size="1.27" layer="1" font="vector" ratio="15" rot="R90" align="bottom-center">v01</text>
+<text x="1.905" y="15.748" size="1.27" layer="1" font="vector" ratio="15" rot="R90" align="bottom-center">v10</text>
 <circle x="2.54" y="22.86" radius="3.048" width="0.254" layer="41"/>
 <circle x="22.86" y="22.86" radius="3.048" width="0.254" layer="41"/>
@@
 </signal>
 </signals>
-<errors>
-</errors>
 </board>
 </drawing>

Commit message: Updated to v10 for release
Parts:
- moved R1 0.25 mm to (18.8, 7.62)
Routing:
- net SCL: track 13.0 -> 12.5 mm
Changed lines of the file:
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@@
 <?xml version="1.0" encoding="utf-8"?>
 <!DOCTYPE eagle SYSTEM "eagle.dtd">
-<eagle version="6.4">
+<eagle version="6.3">
 <drawing>
 <settings>
@@
 <elements>
 <element name="FRAME1" library="SparkFun-Aesthetics" package="CREATIVE_COMMONS" value="FRAME-LETTER" x="-77.47" y="11.43"/>
-<element name="R1" library="SparkFun-Resistors" package="0603-RES" value="1K" x="19.05" y="7.62" rot="R90">
-<attribute name="PROD_ID" value="RES-07856" x="48.26" y="50.8" size="1.778" layer="27" rot="R90" display="off"/>
+<element name="R1" library="SparkFun-Resistors" package="0603-RES" value="1K" x="18.796" y="7.62" rot="R90">
+<attribute name="PROD_ID" value="RES-07856" x="48.006" y="50.8" size="1.778" layer="27" rot="R90" display="off"/>
 </element>
 <element name="R2" library="SparkFun-Resistors" package="0603-RES" value="1K" x="20.32" y="7.62" rot="R90">
@@
 <contactref element="J7" pad="5"/>
 <contactref element="J7" pad="6"/>
-<wire x1="19.05" y1="6.77" x2="19.05" y2="5.461" width="0.254" layer="1"/>
-<wire x1="19.05" y1="5.461" x2="18.796" y2="5.207" width="0.254" layer="1"/>
-<wire x1="18.796" y1="5.207" x2="15.367" y2="5.207" width="0.254" layer="1"/>
+<wire x1="18.796" y1="6.77" x2="18.796" y2="5.461" width="0.254" layer="1"/>
+<wire x1="18.796" y1="5.461" x2="18.542" y2="5.207" width="0.254" layer="1"/>
+<wire x1="18.542" y1="5.207" x2="15.367" y2="5.207" width="0.254" layer="1"/>
 <wire x1="15.367" y1="5.207" x2="15.24" y2="5.08" width="0.254" layer="1"/>
 <wire x1="17.51" y1="9.3205" x2="17.51" y2="7.128" width="0.254" layer="1"/>
 <wire x1="17.51" y1="7.128" x2="17.868" y2="6.77" width="0.254" layer="1"/>
-<wire x1="19.05" y1="6.77" x2="17.868" y2="6.77" width="0.254" layer="1"/>
+<wire x1="18.796" y1="6.77" x2="17.868" y2="6.77" width="0.254" layer="1"/>
 <wire x1="15.24" y1="5.08" x2="15.24" y2="3.81" width="0.254" layer="1"/>
 <wire x1="15.24" y1="3.81" x2="15.24" y2="1.27" width="0.254" layer="1"/>

Commit message: Production Readied
Parts:
- added FID1, FID2: FIDUCIALUFIDUCIAL, SparkFun-Aesthetics:MICRO-FIDUCIAL
Changed lines of the file:
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@@
 <?xml version="1.0" encoding="utf-8"?>
 <!DOCTYPE eagle SYSTEM "eagle.dtd">
-<eagle version="6.3">
+<eagle version="6.4">
 <drawing>
 <settings>
@@
 <setting verticaltext="up"/>
 </settings>
-<grid distance="0.05" unitdist="inch" unit="inch" style="lines" multiple="1" display="yes" altdistance="0.005" altunitdist="inch" altunit="inch"/>
+<grid distance="0.05" unitdist="inch" unit="inch" style="lines" multiple="1" display="yes" altdistance="0.01" altunitdist="inch" altunit="inch"/>
 <layers>
 <layer number="1" name="Top" color="4" fill="1" visible="yes" active="yes"/>
-<layer number="2" name="Route2" color="1" fill="3" visible="no" active="yes"/>
-<layer number="15" name="Route15" color="4" fill="6" visible="no" active="yes"/>
+<layer number="2" name="Route2" color="1" fill="3" visible="yes" active="yes"/>
+<layer number="15" name="Route15" color="4" fill="6" visible="yes" active="yes"/>
 <layer number="16" name="Bottom" color="1" fill="1" visible="yes" active="yes"/>
 <layer number="17" name="Pads" color="2" fill="1" visible="yes" active="yes"/>
 <layer number="18" name="Vias" color="2" fill="1" visible="yes" active="yes"/>
 <layer number="19" name="Unrouted" color="6" fill="1" visible="yes" active="yes"/>
-<layer number="20" name="Dimension" color="15" fill="1" visible="yes" active="yes"/>
-<layer number="21" name="tPlace" color="16" fill="1" visible="yes" active="yes"/>
-<layer number="22" name="bPlace" color="14" fill="1" visible="yes" active="yes"/>
+<layer number="20" name="Dimension" color="6" fill="1" visible="yes" active="yes"/>
+<layer number="21" name="tPlace" color="6" fill="1" visible="yes" active="yes"/>
+<layer number="22" name="bPlace" color="6" fill="1" visible="yes" active="yes"/>
 <layer number="23" name="tOrigins" color="15" fill="1" visible="yes" active="yes"/>
 <layer number="24" name="bOrigins" color="15" fill="1" visible="yes" active="yes"/>
-<layer number="25" name="tNames" color="7" fill="1" visible="no" active="yes"/>
-<layer number="26" name="bNames" color="7" fill="1" visible="no" active="yes"/>
-<layer number="27" name="tValues" color="7" fill="1" visible="no" active="yes"/>
-<layer number="28" name="bValues" color="7" fill="1" visible="no" active="yes"/>
-<layer number="29" name="tStop" color="7" fill="3" visible="no" active="yes"/>
-<layer number="30" name="bStop" color="7" fill="6" visible="no" active="yes"/>
-<layer number="31" name="tCream" color="7" fill="4" visible="no" active="yes"/>
-<layer number="32" name="bCream" color="7" fill="5" visible="no" active="yes"/>
-<layer number="39" name="tKeepout" color="4" fill="11" visible="no" active="yes"/>
-<layer number="40" name="bKeepout" color="1" fill="11" visible="no" active="yes"/>
-<layer number="41" name="tRestrict" color="4" fill="10" visible="no" active="yes"/>
-<layer number="42" name="bRestrict" color="1" fill="10" visible="no" active="yes"/>
-<layer number="43" name="vRestrict" color="2" fill="10" visible="no" active="yes"/>
-<layer number="44" name="Drills" color="7" fill="1" visible="no" active="yes"/>
+<layer number="25" name="tNames" color="7" fill="1" visible="yes" active="yes"/>
+<layer number="26" name="bNames" color="7" fill="1" visible="yes" active="yes"/>
+<layer number="27" name="tValues" color="7" fill="1" visible="yes" active="yes"/>
+<layer number="28" name="bValues" color="7" fill="1" visible="yes" active="yes"/>
+<layer number="29" name="tStop" color="7" fill="3" visible="yes" active="yes"/>
+<layer number="30" name="bStop" color="7" fill="6" visible="yes" active="yes"/>
+<layer number="31" name="tCream" color="7" fill="4" visible="yes" active="yes"/>
+<layer number="32" name="bCream" color="7" fill="5" visible="yes" active="yes"/>
+<layer number="39" name="tKeepout" color="4" fill="11" visible="yes" active="yes"/>
+<layer number="40" name="bKeepout" color="1" fill="11" visible="yes" active="yes"/>
+<layer number="41" name="tRestrict" color="4" fill="10" visible="yes" active="yes"/>
+<layer number="42" name="bRestrict" color="1" fill="10" visible="yes" active="yes"/>
+<layer number="43" name="vRestrict" color="2" fill="10" visible="yes" active="yes"/>
+<layer number="44" name="Drills" color="7" fill="1" visible="yes" active="yes"/>
 <layer number="45" name="Holes" color="7" fill="1" visible="yes" active="yes"/>
-<layer number="46" name="Milling" color="3" fill="1" visible="no" active="yes"/>
+<layer number="46" name="Milling" color="3" fill="1" visible="yes" active="yes"/>
 <layer number="51" name="tDocu" color="6" fill="1" visible="yes" active="yes"/>
-<layer number="52" name="bDocu" color="7" fill="1" visible="no" active="yes"/>
+<layer number="52" name="bDocu" color="7" fill="1" visible="yes" active="yes"/>
 <layer number="3" name="Route3" color="4" fill="3" visible="no" active="no"/>
 <layer number="4" name="Route4" color="1" fill="4" visible="no" active="no"/>
@@
 <element name="LOGO1" library="SparkFun-Aesthetics" package="SFE-LOGO-FLAME" value="LOGO-SFESK" x="7.62" y="19.05"/>
 <element name="LOGO3" library="SparkFun-Aesthetics" package="SFE-LOGO-FLAME" value="LOGO-SFESK" x="6.35" y="21.59" rot="MR90"/>
+<element name="FID1" library="SparkFun-Aesthetics" package="MICRO-FIDUCIAL" value="FIDUCIALUFIDUCIAL" x="0.762" y="24.638"/>
+<element name="FID2" library="SparkFun-Aesthetics" package="MICRO-FIDUCIAL" value="FIDUCIALUFIDUCIAL" x="24.638" y="0.762"/>
 </elements>
 <signals>
